Commit message: Updated robot model to latest one

File: share/urdf/pepper.urdf (robot description, URDF)
Before this commit: robot JulietteY20MP, 84 links, 83 joints
Links:
- removed link ImuBaseGyrometer_frame
- link Hip: geometry collision mesh filename=package://pepper_description/meshes/HipRoll_0.10.stl scale=0.1 0.1 0.1; visual mesh filename=package://pepper_description/meshes/HipRoll.dae scale=0.1 0.1 0.1
- link Pelvis: geometry collision mesh filename=package://pepper_description/meshes/HipPitch_0.10.stl scale=0.1 0.1 0.1; visual mesh filename=package://pepper_description/meshes/HipPitch.dae scale=0.1 0.1 0.1
- link torso: geometry collision mesh filename=package://pepper_description/meshes/Torso_0.10.stl scale=0.1 0.1 0.1; visual mesh filename=package://pepper_description/meshes/Torso.dae scale=0.1 0.1 0.1
Joints:
- removed joint GyrometerBase_sensor_fixedjoint
- joint AccelerometerBase_sensor_fixedjoint: origin xyz=0 0 -0.3 rpy=0 0 0 -> xyz=0.0147 -0.0017 -0.26319 rpy=0 0 0
- joint CameraBottom_sensor_fixedjoint: origin xyz=0.0936 0 0.0616 rpy=0 0.698132 0 -> xyz=0.09262 0 0.06177 rpy=0 0.698132 0
- joint CameraTop_sensor_fixedjoint: origin xyz=0.0868 0 0.1631 rpy=0 0 0 -> xyz=0.08601 0 0.16284 rpy=0 0 0
- joint HeadYaw: origin xyz=-0.038 0 0.1699 rpy=0 0 0 -> xyz=-0.038 0 0.3089 rpy=0 0 0
- joint HipPitch: child Pelvis -> Hip; origin xyz=0 0 -0.079 rpy=0 0 0 -> xyz=0 0 0.268 rpy=0 0 0; parent Hip -> Pelvis
- joint HipRoll: child Hip -> torso; origin xyz=2e-05 0 -0.139 rpy=0 0 0 -> xyz=0 0 0.079 rpy=0 0 0; parent torso -> Hip
- joint KneePitch: child Tibia -> Pelvis; origin xyz=0 0 -0.268 rpy=0 0 0 -> xyz=0 0 0 rpy=0 0 0; parent Pelvis -> Tibia
- joint LShoulderPitch: origin xyz=-0.057 0.14974 0.08682 rpy=0 0 0 -> xyz=-0.057 0.14974 0.22582 rpy=0 0 0
- joint LaserSensor/Front_sensor_fixedjoint: origin xyz=0.0562 0 -0.0692 rpy=0 0.349044 0 -> xyz=0.0562 0 -0.0692 rpy=0 0.349066 0
- joint LaserSensor/Left_sensor_fixedjoint: origin xyz=-0.018 0.0899 -0.0759 rpy=8.34035e-09 0.191982 1.5708 -> xyz=-0.018 0.0899 -0.0759 rpy=0 0.349066 1.5708
- joint LaserSensor/Right_sensor_fixedjoint: origin xyz=-0.018 -0.0899 -0.0759 rpy=4.08851e-07 0.191857 -1.60746 -> xyz=-0.018 -0.0899 -0.0759 rpy=0 0.349066 -1.5708
- joint LaserSensor/Shovel_sensor_fixedjoint: origin xyz=0.0562 0 -0.0692 rpy=0 0.349044 0 -> xyz=0.0562 0 -0.0692 rpy=0 0.349066 0
- joint LaserSensor/VerticalLeft_sensor_fixedjoint: origin xyz=0.0562 0 -0.0692 rpy=0 0.349044 0 -> xyz=0.0562 0 -0.0692 rpy=0 0.349066 0
- joint LaserSensor/VerticalRight_sensor_fixedjoint: origin xyz=0.0562 0 -0.0692 rpy=0 0.349044 0 -> xyz=0.0562 0 -0.0692 rpy=0 0.349066 0
- joint RShoulderPitch: origin xyz=-0.057 -0.14974 0.08682 rpy=0 0 0 -> xyz=-0.057 -0.14974 0.22582 rpy=0 0 0
- joint base_footprint_joint: child base_footprint -> Tibia; origin xyz=0 0 -0.334 rpy=0 0 0 -> xyz=0 0 0.334 rpy=0 0 0; parent Tibia -> base_footprint
- joint base_link_fixedjoint: child torso -> base_link; parent base_link -> torso

Commit message: Update URDF with the joints rotating in the correct direction

File: share/urdf/pepper.urdf (robot description, URDF)
Before this commit: robot JulietteY20MP, 83 links, 82 joints
Joints:
- joint HipPitch: axis 0 1.0 0 -> 0 -1.0 0
- joint HipRoll: axis 1.0 0 0 -> -1.0 0 0
- joint KneePitch: axis 0 1.0 0 -> 0 -1.0 0
